Commit message: wip

File: src/kinematics/ur20.urdf (robot description, URDF)
Before this commit: robot ur20, 9 links, 7 joints
Links:
- added link flange
- link base_link_inertia: mass None -> 4.0; geometry collision mesh filename=package://ur_description/meshes/ur20/collision/base.stl; visual mesh filename=package://ur_description/meshes/ur20/visual/base.dae
- link forearm_link: mass None -> 7.879; geometry collision mesh filename=package://ur_description/meshes/ur20/collision/forearm.stl; visual mesh filename=package://ur_description/meshes/ur20/visual/forearm.dae
- link shoulder_link: mass None -> 16.343; geometry collision mesh filename=package://ur_description/meshes/ur20/collision/shoulder.stl; visual mesh filename=package://ur_description/meshes/ur20/visual/shoulder.dae
- link upper_arm_link: mass None -> 29.632; geometry collision mesh filename=package://ur_description/meshes/ur20/collision/upperarm.stl; visual mesh filename=package://ur_description/meshes/ur20/visual/upperarm.dae
- link wrist_1_link: mass None -> 3.054; geometry collision mesh filename=package://ur_description/meshes/ur20/collision/wrist1.stl; visual mesh filename=package://ur_description/meshes/ur20/visual/wrist1.dae
- link wrist_2_link: mass None -> 3.126; geometry collision mesh filename=package://ur_description/meshes/ur20/collision/wrist2.stl; visual mesh filename=package://ur_description/meshes/ur20/visual/wrist2.dae
- link wrist_3_link: mass None -> 0.926; geometry collision mesh filename=package://ur_description/meshes/ur20/collision/wrist3.stl; visual mesh filename=package://ur_description/meshes/ur20/visual/wrist3.dae
Joints:
- added joint base_joint: type fixed, parent world, child base_link, origin xyz=0 0 0 rpy=0 0 0
- added joint wrist_3-flange: type fixed, parent wrist_3_link, child flange, origin xyz=0 0 0 rpy=0 -1.5707963267948966 -1.5707963267948966
- joint base_link-base_link_inertia: origin xyz=0 0 0 rpy=0 0 0 -> xyz=0 0 0 rpy=0 0 3.141592653589793
